File: KiCad/HotAirGun.sch (KiCad schematic (older format))
At the start: 22 parts, among them J4 Arduino_Nano_Header, Q2 SI2308, SW1 Rotary_Encoder, U1 MAX31855K

Commit message: SOD123 diodes
Parts:
- D1, D2: footprint Diodes_SMD:D_SOD-523 -> Diodes_SMD:D_SOD-123F
Changed lines of the file:
@@
 F 0 "D1" H 2850 5250 50  0000 C CNN
 F 1 "1n4148w" H 2850 5050 50  0000 C CNN
-F 2 "Diodes_SMD:D_SOD-523" H 2850 5150 50  0001 C CNN
+F 2 "Diodes_SMD:D_SOD-123F" H 2850 5150 50  0001 C CNN
 F 3 "" H 2850 5150 50  0001 C CNN
 	1    2850 5150
@@
 F 0 "D2" H 2850 5650 50  0000 C CNN
 F 1 "1n4148w" H 2850 5450 50  0000 C CNN
-F 2 "Diodes_SMD:D_SOD-523" H 2850 5550 50  0001 C CNN
+F 2 "Diodes_SMD:D_SOD-123F" H 2850 5550 50  0001 C CNN
 F 3 "" H 2850 5550 50  0001 C CNN
 	1    2850 5550
