File: KiCad/HotAirGun.kicad_pcb (KiCad board)
At the start: 2 copper layers, 49.8 x 17.6 mm, 22 parts, among them J4 Arduino_Nano_Header, Q2 SI2308, SW1 Rotary_Encoder, U1 MAX31855K

Commit message: Some texts added
Other:
- board text added: "Heat+"
- board text added: "Heat-"
Changed lines of the file:
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@@
     (area 123.224999 118.424999 173.175001 136.175001)
     (thickness 1.6)
-    (drawings 7)
+    (drawings 9)
     (tracks 148)
     (zones 0)
@@
       (net 20 "Net-(Heater_pos1-Pad1)"))
   )
+  (gr_text Heat- (at 126.9 122.5) (layer B.SilkS)
+    (effects (font (size 1.5 1.5) (thickness 0.3)) (justify mirror))
+  )
+  (gr_text Heat+ (at 127.1 132.2) (layer B.SilkS)
+    (effects (font (size 1.5 1.5) (thickness 0.3)) (justify mirror))
+  )
   (gr_text V1.0 (at 157.96 132.49) (layer F.SilkS)
     (effects (font (size 1.2 1.2) (thickness 0.2)))
@@
   (segment (start 143.92 132.28) (end 143.83 132.37) (width 0.4) (layer F.Cu) (net 6))
   (segment (start 159.09 134.99) (end 159.09 133.91) (width 0.4) (layer B.Cu) (net 6))
-  (segment (start 152.97 130.96) (end 143.92 130.96) (width 0.4) (layer F.Cu) (net 6) (status 800000))
+  (segment (start 152.97 130.96) (end 143.92 130.96) (width 0.4) (layer F.Cu) (net 6))
   (segment (start 154.09 132.19) (end 152.97 130.96) (width 0.4) (layer F.Cu) (net 6))
   (via (at 154.09 132.19) (size 0.9) (drill 0.5) (layers F.Cu B.Cu) (net 6))
@@
   (via (at 149.99 128.08) (size 0.9) (drill 0.5) (layers F.Cu B.Cu) (net 13))
   (segment (start 155.39 123.33) (end 154.74 123.33) (width 0.4) (layer F.Cu) (net 13))
-  (segment (start 146.39 131.68) (end 146.39 134.99) (width 0.4) (layer B.Cu) (net 13) (status 800000))
+  (segment (start 146.39 131.68) (end 146.39 134.99) (width 0.4) (layer B.Cu) (net 13))
   (segment (start 156.84 126.33) (end 156.84 127.78) (width 0.4) (layer F.Cu) (net 14))
   (segment (start 156.84 127.78) (end 156.79 127.83) (width 0.4) (layer F.Cu) (net 14))
@@
   (via (at 152.26 128.14) (size 0.9) (drill 0.5) (layers F.Cu B.Cu) (net 15))
   (segment (start 155.39 127.83) (end 152.57 127.83) (width 0.4) (layer F.Cu) (net 15))
-  (segment (start 148.93 131.47) (end 148.93 134.99) (width 0.4) (layer B.Cu) (net 15) (status 800000))
+  (segment (start 148.93 131.47) (end 148.93 134.99) (width 0.4) (layer B.Cu) (net 15))
   (segment (start 167.3 130.9) (end 168.34 130.9) (width 0.4) (layer F.Cu) (net 16))
   (segment (start 169.94 129.3) (end 171.5 129.3) (width 0.4) (layer F.Cu) (net 16))
@@
   (segment (start 146.39 119.75) (end 146.39 122.02) (width 0.4) (layer F.Cu) (net 17))
   (segment (start 146.39 122.02) (end 146.4 122.03) (width 0.4) (layer F.Cu) (net 17))
-  (segment (start 161.7 131.55) (end 155.43 131.55) (width 0.4) (layer F.Cu) (net 18) (status 400000))
-  (segment (start 144.88 133.96) (end 143.85 134.99) (width 0.4) (layer B.Cu) (net 18) (status 800000))
+  (segment (start 161.7 131.55) (end 155.43 131.55) (width 0.4) (layer F.Cu) (net 18))
+  (segment (start 144.88 133.96) (end 143.85 134.99) (width 0.4) (layer B.Cu) (net 18))
   (segment (start 144.88 130.34) (end 144.88 133.96) (width 0.4) (layer B.Cu) (net 18))
   (segment (start 145.34 129.88) (end 144.88 130.34) (width 0.4) (layer B.Cu) (net 18))
@@
   (via (at 157.88 128.6) (size 0.9) (drill 0.5) (layers F.Cu B.Cu) (net 19))
   (segment (start 159.5 126.235) (end 158.685 126.235) (width 0.4) (layer F.Cu) (net 19))
-  (segment (start 151.47 131.28) (end 151.47 134.99) (width 0.4) (layer B.Cu) (net 19) (status 800000))
+  (segment (start 151.47 131.28) (end 151.47 134.99) (width 0.4) (layer B.Cu) (net 19))
   (segment (start 153.31 129.44) (end 151.47 131.28) (width 0.4) (layer B.Cu) (net 19))
   (segment (start 157.04 129.44) (end 153.31 129.44) (width 0.4) (layer B.Cu) (net 19))

Commit message: Final adjustments
Routing:
- net GND: track 4.71 -> 8.02 mm, vias 2 -> 3
- net VCC: track 28.8 -> 29.8 mm
Other:
- rule pad_to_mask_clearance: 0.2 -> 0.1
Changed lines of the file:
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@@
     (thickness 1.6)
     (drawings 9)
-    (tracks 148)
+    (tracks 155)
     (zones 0)
     (modules 22)
@@
     (pad_size 1.524 1.524)
     (pad_drill 0.762)
-    (pad_to_mask_clearance 0.2)
+    (pad_to_mask_clearance 0.1)
     (aux_axis_origin 0 0)
     (visible_elements 7FFFFF7F)
@@
   (gr_line (start 173.1 136.1) (end 173.1 118.5) (angle 90) (layer Edge.Cuts) (width 0.15))
   (gr_line (start 123.3 118.5) (end 123.3 136.1) (angle 90) (layer Edge.Cuts) (width 0.15))
+  (segment (start 162.35 127.5) (end 162.35 125.25) (width 0.4) (layer F.Cu) (net 1))
+  (segment (start 162.915 127.505) (end 162.35 127.5) (width 0.4) (layer F.Cu) (net 1))
+  (via (at 162.35 127.5) (size 1.5) (drill 0.8) (layers F.Cu B.Cu) (net 1))
   (segment (start 164.9 127.505) (end 162.915 127.505) (width 0.4) (layer F.Cu) (net 1))
-  (via (at 162.37 126.96) (size 1.5) (drill 0.8) (layers F.Cu B.Cu) (net 1))
-  (segment (start 162.915 127.505) (end 162.37 126.96) (width 0.4) (layer F.Cu) (net 1))
+  (via (at 161.45 124.35) (size 1.5) (drill 0.8) (layers F.Cu B.Cu) (net 1))
+  (segment (start 162.35 125.25) (end 161.45 124.35) (width 0.4) (layer F.Cu) (net 1))
   (segment (start 165.3 131.85) (end 166.02 131.85) (width 0.4) (layer F.Cu) (net 1))
   (via (at 166.89 132.72) (size 1.5) (drill 0.8) (layers F.Cu B.Cu) (net 1))
@@
   (segment (start 155.17 121.33) (end 153.9 121.33) (width 0.4) (layer F.Cu) (net 3))
   (segment (start 156.55 119.4) (end 156.55 119.75) (width 0.4) (layer F.Cu) (net 3))
-  (segment (start 164.17 119.75) (end 164.17 122.91) (width 0.4) (layer B.Cu) (net 4))
-  (segment (start 142.27 129.38) (end 141.2 129.38) (width 0.4) (layer B.Cu) (net 4))
+  (segment (start 144.73 126.92) (end 148.78 126.92) (width 0.4) (layer B.Cu) (net 4))
+  (segment (start 164.17 123.86) (end 161.11 126.92) (width 0.4) (layer B.Cu) (net 4))
   (segment (start 144.73 126.92) (end 142.27 129.38) (width 0.4) (layer B.Cu) (net 4))
-  (segment (start 160.16 126.92) (end 144.73 126.92) (width 0.4) (layer B.Cu) (net 4))
-  (segment (start 164.17 122.91) (end 160.16 126.92) (width 0.4) (layer B.Cu) (net 4))
+  (segment (start 141.2 129.38) (end 142.27 129.38) (width 0.4) (layer B.Cu) (net 4))
+  (segment (start 164.17 123.86) (end 164.17 119.75) (width 0.4) (layer B.Cu) (net 4) (status 800000))
+  (segment (start 153.62 126.92) (end 161.11 126.92) (width 0.4) (layer B.Cu) (net 4))
+  (segment (start 153.1 126.4) (end 153.62 126.92) (width 0.4) (layer B.Cu) (net 4))
+  (segment (start 149.3 126.4) (end 153.1 126.4) (width 0.4) (layer B.Cu) (net 4))
+  (segment (start 148.78 126.92) (end 149.3 126.4) (width 0.4) (layer B.Cu) (net 4))
   (via (at 141.2 129.38) (size 0.9) (drill 0.5) (layers F.Cu B.Cu) (net 4))
   (segment (start 141.2 129.38) (end 141.21 129.39) (width 0.4) (layer B.Cu) (net 4))
